File: Carte Elec/VentilationLignade/VentilationLignade.sch (KiCad schematic (older format))
At the start: 27 parts, among them P1 CONN_4, P10 CONN_5, P11 CONN_5, P12 CONN_7X2, P13 CONN_2, P14 CONN_13X2, P15 CONN_2, P16 CONN_7, P17 CONN_2, P18 CONN_4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

Commit message: Ajout Netliste creation Board
Parts:
- removed P14: CONN_13X2, symbol CONN_13X2
- added P14: Teensy_Haut, symbol CONN_13
- added P22: Teensy_Bas, symbol CONN_13
- P1: value CONN_4 -> RelaisBoard1
- P10: value CONN_5 -> SDCard
- P11: value CONN_5 -> Codeur Rotatif
- P12: value CONN_7X2 -> Teensy dessous
- P13: value CONN_2 -> EndStops1
- P15: value CONN_2 -> EndStops2
- P16: value CONN_7 -> Teensy_cote
- P17: value CONN_2 -> Retour 12V
- P18: value CONN_4 -> Masse_12V
- P19: value CONN_2 -> 12V1
- P2: value CONN_5 -> Temp_Ext
- P20: value CONN_2 -> 12V2
- P21: value CONN_2 -> 12V_1et2
- P3: value CONN_4 -> RelaisBoard2
- P4: value CONN_5 -> Temp_Int
- P5: value CONN_4 -> RelaisBoard3
- P6: value CONN_5 -> Temp_Chem
- P7: value CONN_4 -> RelaisBoard4
- P8: value CONN_4 -> RelaisBoard5
- P9: value CONN_9 -> TFT
- SW1: value SWITCH_INV -> Reset_Push
- SW2: value SWITCH_INV -> BackLight_On/ff
Changed lines of the file:
@@
 P 800 7450
 F 0 "P1" V 750 7450 50  0000 C CNN
-F 1 "CONN_4" V 850 7450 50  0000 C CNN
+F 1 "RelaisBoard1" V 850 7450 50  0000 C CNN
 F 2 "" H 800 7450 60  0000 C CNN
 F 3 "" H 800 7450 60  0000 C CNN
@@
 P 1350 7450
 F 0 "P3" V 1300 7450 50  0000 C CNN
-F 1 "CONN_4" V 1400 7450 50  0000 C CNN
+F 1 "RelaisBoard2" V 1400 7450 50  0000 C CNN
 F 2 "" H 1350 7450 60  0000 C CNN
 F 3 "" H 1350 7450 60  0000 C CNN
@@
 P 1900 7450
 F 0 "P5" V 1850 7450 50  0000 C CNN
-F 1 "CONN_4" V 1950 7450 50  0000 C CNN
+F 1 "RelaisBoard3" V 1950 7450 50  0000 C CNN
 F 2 "" H 1900 7450 60  0000 C CNN
 F 3 "" H 1900 7450 60  0000 C CNN
@@
 P 2450 7450
 F 0 "P7" V 2400 7450 50  0000 C CNN
-F 1 "CONN_4" V 2500 7450 50  0000 C CNN
+F 1 "RelaisBoard4" V 2500 7450 50  0000 C CNN
 F 2 "" H 2450 7450 60  0000 C CNN
 F 3 "" H 2450 7450 60  0000 C CNN
@@
 P 3000 7450
 F 0 "P8" V 2950 7450 50  0000 C CNN
-F 1 "CONN_4" V 3050 7450 50  0000 C CNN
+F 1 "RelaisBoard5" V 3050 7450 50  0000 C CNN
 F 2 "" H 3000 7450 60  0000 C CNN
 F 3 "" H 3000 7450 60  0000 C CNN
@@
 P 10650 800
 F 0 "P19" V 10600 800 40  0000 C CNN
-F 1 "CONN_2" V 10700 800 40  0000 C CNN
+F 1 "12V1" V 10700 800 40  0000 C CNN
 F 2 "" H 10650 800 60  0000 C CNN
 F 3 "" H 10650 800 60  0000 C CNN
@@
 P 10650 1300
 F 0 "P20" V 10600 1300 40  0000 C CNN
-F 1 "CONN_2" V 10700 1300 40  0000 C CNN
+F 1 "12V2" V 10700 1300 40  0000 C CNN
 F 2 "" H 10650 1300 60  0000 C CNN
 F 3 "" H 10650 1300 60  0000 C CNN
@@
 P 10850 6600
 F 0 "P21" V 10800 6600 40  0000 C CNN
-F 1 "CONN_2" V 10900 6600 40  0000 C CNN
+F 1 "12V_1et2" V 10900 6600 40  0000 C CNN
 F 2 "" H 10850 6600 60  0000 C CNN
 F 3 "" H 10850 6600 60  0000 C CNN
@@
 P 9900 6600
 F 0 "P18" V 9850 6600 50  0000 C CNN
-F 1 "CONN_4" V 9950 6600 50  0000 C CNN
+F 1 "Masse_12V" V 9950 6600 50  0000 C CNN
 F 2 "" H 9900 6600 60  0000 C CNN
 F 3 "" H 9900 6600 60  0000 C CNN
@@
 P 1050 1050
 F 0 "P2" V 1000 1050 50  0000 C CNN
-F 1 "CONN_5" V 1100 1050 50  0000 C CNN
+F 1 "Temp_Ext" V 1100 1050 50  0000 C CNN
 F 2 "" H 1050 1050 60  0000 C CNN
 F 3 "" H 1050 1050 60  0000 C CNN
@@
 P 1650 1050
 F 0 "P4" V 1600 1050 50  0000 C CNN
-F 1 "CONN_5" V 1700 1050 50  0000 C CNN
+F 1 "Temp_Int" V 1700 1050 50  0000 C CNN
 F 2 "" H 1650 1050 60  0000 C CNN
 F 3 "" H 1650 1050 60  0000 C CNN
@@
 P 2250 1050
 F 0 "P6" V 2200 1050 50  0000 C CNN
-F 1 "CONN_5" V 2300 1050 50  0000 C CNN
+F 1 "Temp_Chem" V 2300 1050 50  0000 C CNN
 F 2 "" H 2250 1050 60  0000 C CNN
 F 3 "" H 2250 1050 60  0000 C CNN
@@
 P 5250 1050
 F 0 "P11" V 5200 1050 50  0000 C CNN
-F 1 "CONN_5" V 5300 1050 50  0000 C CNN
+F 1 "Codeur Rotatif" V 5300 1050 50  0000 C CNN
 F 2 "" H 5250 1050 60  0000 C CNN
 F 3 "" H 5250 1050 60  0000 C CNN
@@
 P 4350 1050
 F 0 "P10" V 4300 1050 50  0000 C CNN
-F 1 "CONN_5" V 4400 1050 50  0000 C CNN
+F 1 "SDCard" V 4400 1050 50  0000 C CNN
 F 2 "" H 4350 1050 60  0000 C CNN
 F 3 "" H 4350 1050 60  0000 C CNN
@@
 P 3350 1050
 F 0 "P9" V 3300 1050 60  0000 C CNN
-F 1 "CONN_9" V 3400 1050 60  0000 C CNN
+F 1 "TFT" V 3400 1050 60  0000 C CNN
 F 2 "" H 3350 1050 60  0000 C CNN
 F 3 "" H 3350 1050 60  0000 C CNN
@@
 P 7200 1050
 F 0 "P13" V 7150 1050 40  0000 C CNN
-F 1 "CONN_2" V 7250 1050 40  0000 C CNN
+F 1 "EndStops1" V 7250 1050 40  0000 C CNN
 F 2 "" H 7200 1050 60  0000 C CNN
 F 3 "" H 7200 1050 60  0000 C CNN
@@
 P 7900 1050
 F 0 "P15" V 7850 1050 40  0000 C CNN
-F 1 "CONN_2" V 7950 1050 40  0000 C CNN
+F 1 "EndStops2" V 7950 1050 40  0000 C CNN
 F 2 "" H 7900 1050 60  0000 C CNN
 F 3 "" H 7900 1050 60  0000 C CNN
@@
 P 3650 3250
 F 0 "SW2" H 3450 3400 50  0000 C CNN
-F 1 "SWITCH_INV" H 3500 3100 50  0000 C CNN
+F 1 "BackLight_On/ff" H 3500 3100 50  0000 C CNN
 F 2 "~" H 3650 3250 60  0000 C CNN
 F 3 "~" H 3650 3250 60  0000 C CNN
@@
 P 3250 3050
 F 0 "SW1" H 3050 3200 50  0000 C CNN
-F 1 "SWITCH_INV" H 3100 2900 50  0000 C CNN
+F 1 "Reset_Push" H 3100 2900 50  0000 C CNN
 F 2 "~" H 3250 3050 60  0000 C CNN
 F 3 "~" H 3250 3050 60  0000 C CNN
@@
 $EndComp
 $Comp
-L CONN_13X2 P14
-U 1 1 55ECA18B
-P 7350 5150
-F 0 "P14" H 7350 5850 60  0000 C CNN
-F 1 "CONN_13X2" V 7350 5150 50  0000 C CNN
-F 2 "" H 7350 5150 60  0000 C CNN
-F 3 "" H 7350 5150 60  0000 C CNN
-	1    7350 5150
-	0    -1   -1   0
-$EndComp
-$Comp
 L CONN_7 P16
 U 1 1 55ECA19A
 P 8200 5150
 F 0 "P16" V 8170 5150 60  0000 C CNN
-F 1 "CONN_7" V 8270 5150 60  0000 C CNN
+F 1 "Teensy_cote" V 8270 5150 60  0000 C CNN
 F 2 "" H 8200 5150 60  0000 C CNN
 F 3 "" H 8200 5150 60  0000 C CNN
@@
 P 5250 5150
 F 0 "P12" H 5250 5550 60  0000 C CNN
-F 1 "CONN_7X2" V 5250 5150 60  0000 C CNN
+F 1 "Teensy dessous" V 5250 5150 60  0000 C CNN
 F 2 "" H 5250 5150 60  0000 C CNN
 F 3 "" H 5250 5150 60  0000 C CNN
@@
 P 8900 1050
 F 0 "P17" V 8850 1050 40  0000 C CNN
-F 1 "CONN_2" V 8950 1050 40  0000 C CNN
+F 1 "Retour 12V" V 8950 1050 40  0000 C CNN
 F 2 "" H 8900 1050 60  0000 C CNN
 F 3 "" H 8900 1050 60  0000 C CNN
@@
 Wire Notes Line
 	6250 7100 6250 7750
+$Comp
+L CONN_13 P22
+U 1 1 55ECB3C0
+P 7350 5200
+F 0 "P22" V 7300 5700 60  0000 C CNN
+F 1 "Teensy_Bas" V 7300 5200 60  0000 C CNN
+F 2 "" H 7350 5200 60  0000 C CNN
+F 3 "" H 7350 5200 60  0000 C CNN
+	1    7350 5200
+	0    -1   -1   0
+$EndComp
+$Comp
+L CONN_13 P14
+U 1 1 55ECB3CF
+P 7350 5100
+F 0 "P14" V 7300 4600 60  0000 C CNN
+F 1 "Teensy_Haut" V 7300 5100 60  0000 C CNN
+F 2 "" H 7350 5100 60  0000 C CNN
+F 3 "" H 7350 5100 60  0000 C CNN
+	1    7350 5100
+	0    1    1    0
+$EndComp
 $EndSCHEMATC

Commit message: Dessin de carte. Changement des pins pour avoir un truc cohérent au niveau de la carte.
Connections:
- wire segments 196 -> 195
Changed lines of the file:
@@
 Sheet 1 2
 Title ""
-Date "6 sep 2015"
+Date "7 sep 2015"
 Rev ""
 Comp ""
@@
 NoConn ~ 5550 4750
 NoConn ~ 5450 4750
-Text GLabel 6950 6150 0    60   Output ~ 0
+Text GLabel 6600 5900 0    60   Output ~ 0
 BYPASS_1_F
-Text GLabel 6950 6300 0    60   Output ~ 0
+Text GLabel 6600 6050 0    60   Output ~ 0
 BYPASS_1_O
-Text GLabel 6950 6450 0    60   Output ~ 0
+Text GLabel 6600 6200 0    60   Output ~ 0
 BYPASS_2_F
-Text GLabel 6950 6600 0    60   Output ~ 0
+Text GLabel 6600 6350 0    60   Output ~ 0
 BYPASS_2_O
 Text GLabel 8400 6300 2    60   Output ~ 0
@@
 	6750 5550 6750 5750
 Wire Wire Line
-	6950 6150 7150 6150
-Wire Wire Line
-	7150 6150 7150 5550
-Wire Wire Line
-	6950 6300 7250 6300
-Wire Wire Line
-	7250 6300 7250 5550
-Wire Wire Line
-	6950 6450 7350 6450
-Wire Wire Line
-	7350 6450 7350 5550
-Wire Wire Line
-	6950 6600 7450 6600
-Wire Wire Line
-	7450 6600 7450 5550
-Wire Wire Line
 	8400 5900 7950 5900
 Wire Wire Line
@@
 Wire Wire Line
 	7450 3950 7450 4750
-NoConn ~ 7950 4750
 Text GLabel 6550 3650 0    60   Output ~ 0
 TEXT_CS
@@
 	7050 4050 7050 4750
 NoConn ~ 7350 4750
-NoConn ~ 7550 5550
-NoConn ~ 7650 5550
-NoConn ~ 7050 5550
-NoConn ~ 6950 5550
-NoConn ~ 6850 5550
-Text GLabel 4400 6300 0    60   Output ~ 0
+Text GLabel 6600 6650 0    60   Output ~ 0
 VENT_CHEMINEE
-Text GLabel 4400 6150 0    60   Output ~ 0
+Text GLabel 6600 6500 0    60   Output ~ 0
 VENT_CAVE
-Text GLabel 4400 6000 0    60   Output ~ 0
+Text GLabel 7750 6750 2    60   Output ~ 0
 SELECT_VMC
-Text GLabel 4400 5850 0    60   Output ~ 0
+Text GLabel 6600 6800 0    60   Output ~ 0
 12V1_ON
-Text GLabel 4400 5700 0    60   Output ~ 0
+Text GLabel 7750 6550 2    60   Output ~ 0
 12V2_ON
-Wire Wire Line
-	4400 5700 4950 5700
-Wire Wire Line
-	4950 5700 4950 5550
-Wire Wire Line
-	4400 5850 5050 5850
-Wire Wire Line
-	5050 5850 5050 5550
-Wire Wire Line
-	4400 6000 5150 6000
-Wire Wire Line
-	5150 6000 5150 5550
-Wire Wire Line
-	4400 6150 5250 6150
-Wire Wire Line
-	5250 6150 5250 5550
-Wire Wire Line
-	4400 6300 5350 6300
-Wire Wire Line
-	5350 6300 5350 5550
-Text GLabel 4300 4700 0    60   Output ~ 0
+Text GLabel 4300 5550 0    60   Output ~ 0
 SELECT_12V
-Text GLabel 4300 4550 0    60   Input ~ 0
+Text GLabel 8200 4700 2    60   Input ~ 0
 12V_CHECK
+Text GLabel 4300 5700 0    60   Input ~ 0
+ENCODEUR_SW
 Text GLabel 4300 4400 0    60   Input ~ 0
-ENCODEUR_SW
-Text GLabel 4300 4250 0    60   Input ~ 0
 ENCODEUR_A
-Text GLabel 4300 4100 0    60   Input ~ 0
+Text GLabel 4300 5850 0    60   Input ~ 0
 ENCODEUR_B
-Wire Wire Line
-	4300 4700 4950 4700
-Wire Wire Line
-	4950 4700 4950 4750
-Wire Wire Line
-	4300 4550 5050 4550
-Wire Wire Line
-	5050 4550 5050 4750
-Wire Wire Line
-	4300 4400 5150 4400
-Wire Wire Line
-	4300 4250 5250 4250
-Wire Wire Line
-	5250 4250 5250 4750
-Wire Wire Line
-	4300 4100 5350 4100
-Wire Wire Line
-	5350 4100 5350 4750
 $Comp
 L CONN_2 P17
@@
 Wire Wire Line
 	7100 3250 9100 3250
-Wire Wire Line
-	5150 4400 5150 4750
 $Comp
 L +3.3V #PWR030
@@
 	0    1    1    0
 $EndComp
+Wire Wire Line
+	6600 5900 6850 5900
+Wire Wire Line
+	6850 5900 6850 5550
+Wire Wire Line
+	6600 6050 6950 6050
+Wire Wire Line
+	6950 6050 6950 5550
+Wire Wire Line
+	6600 6200 7050 6200
+Wire Wire Line
+	7050 6200 7050 5550
+Wire Wire Line
+	6600 6350 7150 6350
+Wire Wire Line
+	7150 6350 7150 5550
+Wire Wire Line
+	6600 6500 7250 6500
+Wire Wire Line
+	7250 6500 7250 5550
+Wire Wire Line
+	6600 6650 7350 6650
+Wire Wire Line
+	7350 6650 7350 5550
+Wire Wire Line
+	6600 6800 7450 6800
+Wire Wire Line
+	7450 6800 7450 5550
+Wire Wire Line
+	7650 6550 7750 6550
+Wire Wire Line
+	7650 6550 7650 5550
+Wire Wire Line
+	7750 6750 7550 6750
+Wire Wire Line
+	7550 6750 7550 5550
+NoConn ~ 5250 5550
+NoConn ~ 5350 5550
+Wire Wire Line
+	4300 5550 4950 5550
+Wire Wire Line
+	4300 4400 5050 4400
+Wire Wire Line
+	5050 4400 5050 4750
+Wire Wire Line
+	4300 5700 5050 5700
+Wire Wire Line
+	5050 5700 5050 5550
+Wire Wire Line
+	4300 5850 5150 5850
+Wire Wire Line
+	5150 5850 5150 5550
+NoConn ~ 5150 4750
+NoConn ~ 5250 4750
+NoConn ~ 5350 4750
+Wire Wire Line
+	7950 4750 7950 4700
+Wire Wire Line
+	7950 4700 8200 4700
+NoConn ~ 4950 4750
 $EndSCHEMATC

Commit message: Ajout d'un RS232 MAX au cas ou.
Parts:
- added C4, C5, C6, C7, C8: C, ~, symbol C
- added P23: CONN_4, symbol CONN_4
- added R2, R3: R, ~, symbol R
- added U1: MAX232, symbol MAX232
Connections:
- net labels added: RX, TX
- wire segments 195 -> 224
- no-connect marks 19 -> 18
Changed lines of the file:
@@
 Sheet 1 2
 Title ""
-Date "7 sep 2015"
+Date "8 sep 2015"
 Rev ""
 Comp ""
@@
 Text GLabel 8200 4700 2    60   Input ~ 0
 12V_CHECK
-Text GLabel 4300 5700 0    60   Input ~ 0
+Text GLabel 4300 4550 0    60   Input ~ 0
 ENCODEUR_SW
 Text GLabel 4300 4400 0    60   Input ~ 0
@@
 Wire Wire Line
 	5050 4400 5050 4750
-Wire Wire Line
-	4300 5700 5050 5700
-Wire Wire Line
-	5050 5700 5050 5550
-Wire Wire Line
-	4300 5850 5150 5850
-Wire Wire Line
-	5150 5850 5150 5550
-NoConn ~ 5150 4750
 NoConn ~ 5250 4750
 NoConn ~ 5350 4750
@@
 Wire Wire Line
 	7950 4700 8200 4700
-NoConn ~ 4950 4750
+Wire Wire Line
+	4300 4550 4950 4550
+Wire Wire Line
+	4950 4550 4950 4750
+$Comp
+L MAX232 U1
+U 1 1 55EEB4F2
+P 1800 4800
+F 0 "U1" H 1800 5650 70  0000 C CNN
+F 1 "MAX232" H 1800 3950 70  0000 C CNN
+F 2 "" H 1800 4800 60  0000 C CNN
+F 3 "" H 1800 4800 60  0000 C CNN
+	1    1800 4800
+	-1   0    0    -1
+$EndComp
+$Comp
+L C C7
+U 1 1 55EEB60C
+P 2800 4300
+F 0 "C7" H 2800 4400 40  0000 L CNN
+F 1 "C" H 2806 4215 40  0000 L CNN
+F 2 "~" H 2838 4150 30  0000 C CNN
+F 3 "~" H 2800 4300 60  0000 C CNN
+	1    2800 4300
+	1    0    0    -1
+$EndComp
+$Comp
+L C C8
+U 1 1 55EEB61B
+P 2800 4800
+F 0 "C8" H 2800 4900 40  0000 L CNN
+F 1 "C" H 2806 4715 40  0000 L CNN
+F 2 "~" H 2838 4650 30  0000 C CNN
+F 3 "~" H 2800 4800 60  0000 C CNN
+	1    2800 4800
+	1    0    0    -1
+$EndComp
+$Comp
+L CONN_4 P23
+U 1 1 55EEB62A
+P 600 5350
+F 0 "P23" V 550 5350 50  0000 C CNN
+F 1 "CONN_4" V 650 5350 50  0000 C CNN
+F 2 "" H 600 5350 60  0000 C CNN
+F 3 "" H 600 5350 60  0000 C CNN
+	1    600  5350
+	-1   0    0    1
+$EndComp
+Wire Wire Line
+	950  5200 1000 5200
+Wire Wire Line
+	950  5300 1000 5300
+Wire Wire Line
+	950  5400 1000 5400
+Wire Wire Line
+	950  5500 1000 5500
+Wire Wire Line
+	2600 4100 2800 4100
+Wire Wire Line
+	2600 4500 2800 4500
+Wire Wire Line
+	2600 4600 2800 4600
+Wire Wire Line
+	2800 5000 2600 5000
+$Comp
+L GND #PWR038
+U 1 1 55EEBF63
+P 800 4750
+F 0 "#PWR038" H 800 4750 30  0001 C CNN
+F 1 "GND" H 800 4680 30  0001 C CNN
+F 2 "" H 800 4750 60  0000 C CNN
+F 3 "" H 800 4750 60  0000 C CNN
+	1    800  4750
+	1    0    0    -1
+$EndComp
+Wire Wire Line
+	800  4750 800  4700
+Wire Wire Line
+	800  4700 1000 4700
+$Comp
+L +3.3V #PWR039
+U 1 1 55EEC091
+P 800 4050
+F 0 "#PWR039" H 800 4010 30  0001 C CNN
+F 1 "+3.3V" H 800 4160 30  0000 C CNN
+F 2 "" H 800 4050 60  0000 C CNN
+F 3 "" H 800 4050 60  0000 C CNN
+	1    800  4050
+	1    0    0    -1
+$EndComp
+Wire Wire Line
+	800  4050 800  4100
+Wire Wire Line
+	550  4100 1000 4100
+$Comp
+L C C6
+U 1 1 55EF1C27
+P 750 4300
+F 0 "C6" H 750 4400 40  0000 L CNN
+F 1 "C" H 756 4215 40  0000 L CNN
+F 2 "~" H 788 4150 30  0000 C CNN
+F 3 "~" H 750 4300 60  0000 C CNN
+	1    750  4300
+	1    0    0    -1
+$EndComp
+$Comp
+L C C4
+U 1 1 55EF1C37
+P 550 4300
+F 0 "C4" H 550 4400 40  0000 L CNN
+F 1 "C" H 556 4215 40  0000 L CNN
+F 2 "~" H 588 4150 30  0000 C CNN
+F 3 "~" H 550 4300 60  0000 C CNN
+	1    550  4300
+	1    0    0    -1
+$EndComp
+$Comp
+L C C5
+U 1 1 55EF1C46
+P 550 4800
+F 0 "C5" H 550 4900 40  0000 L CNN
+F 1 "C" H 556 4715 40  0000 L CNN
+F 2 "~" H 588 4650 30  0000 C CNN
+F 3 "~" H 550 4800 60  0000 C CNN
+	1    550  4800
+	1    0    0    -1
+$EndComp
+Connection ~ 800  4100
+Connection ~ 750  4100
+Wire Wire Line
+	750  4500 1000 4500
+Wire Wire Line
+	550  4500 550  4600
+Wire Wire Line
+	550  5000 1000 5000
+$Comp
+L GND #PWR040
+U 1 1 55EF2234
+P 650 4600
+F 0 "#PWR040" H 650 4600 30  0001 C CNN
+F 1 "GND" H 650 4530 30  0001 C CNN
+F 2 "" H 650 4600 60  0000 C CNN
+F 3 "" H 650 4600 60  0000 C CNN
+	1    650  4600
+	1    0    0    -1
+$EndComp
+Wire Wire Line
+	550  4550 650  4550
+Wire Wire Line
+	650  4550 650  4600
+Connection ~ 550  4550
+$Comp
+L GND #PWR041
+U 1 1 55EF236C
+P 1700 5800
+F 0 "#PWR041" H 1700 5800 30  0001 C CNN
+F 1 "GND" H 1700 5730 30  0001 C CNN
+F 2 "" H 1700 5800 60  0000 C CNN
+F 3 "" H 1700 5800 60  0000 C CNN
+	1    1700 5800
+	1    0    0    -1
+$EndComp
+$Comp
+L R R2
+U 1 1 55EF237B
+P 1300 5700
+F 0 "R2" V 1380 5700 40  0000 C CNN
+F 1 "R" V 1307 5701 40  0000 C CNN
+F 2 "~" V 1230 5700 30  0000 C CNN
+F 3 "~" H 1300 5700 30  0000 C CNN
+	1    1300 5700
+	0    -1   -1   0
+$EndComp
+Wire Wire Line
+	1050 5700 950  5700
+Wire Wire Line
+	950  5700 950  5500
+Wire Wire Line
+	1550 5700 1700 5700
+Wire Wire Line
+	1700 5700 1700 5800
+$Comp
+L R R3
+U 1 1 55EF267E
+P 3000 5550
+F 0 "R3" V 3080 5550 40  0000 C CNN
+F 1 "R" V 3007 5551 40  0000 C CNN
+F 2 "~" V 2930 5550 30  0000 C CNN
+F 3 "~" H 3000 5550 30  0000 C CNN
+	1    3000 5550
+	1    0    0    -1
+$EndComp
+NoConn ~ 2600 5500
+Wire Wire Line
+	2600 5300 3000 5300
+$Comp
+L GND #PWR042
+U 1 1 55EF27BC
+P 3000 5850
+F 0 "#PWR042" H 3000 5850 30  0001 C CNN
+F 1 "GND" H 3000 5780 30  0001 C CNN
+F 2 "" H 3000 5850 60  0000 C CNN
+F 3 "" H 3000 5850 60  0000 C CNN
+	1    3000 5850
+	1    0    0    -1
+$EndComp
+Wire Wire Line
+	3000 5850 3000 5800
+Text GLabel 2750 5200 2    60   Input ~ 0
+TX
+Wire Wire Line
+	2750 5200 2600 5200
+Text GLabel 2750 5400 2    60   Output ~ 0
+RX
+Wire Wire Line
+	2750 5400 2600 5400
+Text GLabel 4300 6150 0    60   Input ~ 0
+RX
+Wire Wire Line
+	4300 5850 5050 5850
+Wire Wire Line
+	5050 5850 5050 5550
+Wire Wire Line
+	4300 6150 5150 6150
+Wire Wire Line
+	5150 6150 5150 5550
+Text GLabel 4300 4250 0    60   Output ~ 0
+TX
+Wire Wire Line
+	4300 4250 5150 4250
+Wire Wire Line
+	5150 4250 5150 4750
 $EndSCHEMATC

Commit message: Reprise de la carte => Dimensions réduites 50x100mm
Parts:
- removed C6: C, ~, symbol C
- removed P12: Teensy dessous, symbol CONN_7X2
- added P12: Teensy Bottom, symbol CONN_10
- added P24: Temp_PuitC, symbol CONN_5
- P23: value CONN_4 -> Serial
Connections:
- net labels added: TPUIT_CS
- wire segments 224 -> 245
- no-connect marks 18 -> 13
Other:
- moved on the sheet: C1, C2, C3, P10, P11, P13, P15, P17, P19, P2, P20, P23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
