File: Carte Elec/VentilationLignade/Optocouplers.sch (KiCad schematic (older format))
At the start: 35 parts, among them U2 OPTO-TRANSISTOR, U3 OPTO-TRANSISTOR, U4 OPTO-TRANSISTOR, U5 OPTO-TRANSISTOR, U6 OPTO-TRANSISTOR

Commit message: Modif elec et dossier de commande carte
Changed lines of the file:
@@
 Sheet 2 2
 Title ""
-Date "1 oct 2015"
+Date "6 apr 2017"
 Rev ""
 Comp ""
@@
 F 0 "#PWR043" H 4650 2050 30  0001 C CNN
 F 1 "GND" H 4650 1980 30  0001 C CNN
-F 2 "" H 4650 2050 60  0000 C CNN
-F 3 "" H 4650 2050 60  0000 C CNN
+F 2 "" H 4650 2050 60  0001 C CNN
+F 3 "" H 4650 2050 60  0001 C CNN
 	1    4650 2050
 	1    0    0    -1
@@
 F 0 "#PWR044" H 4950 1250 30  0001 C CNN
 F 1 "GND" H 4950 1180 30  0001 C CNN
-F 2 "" H 4950 1250 60  0000 C CNN
-F 3 "" H 4950 1250 60  0000 C CNN
+F 2 "" H 4950 1250 60  0001 C CNN
+F 3 "" H 4950 1250 60  0001 C CNN
 	1    4950 1250
 	1    0    0    -1
@@
 Connection ~ 4700 1150
 Wire Wire Line
-	4650 1750 4650 2050
+	4650 2050 4650 1750
 $Comp
 L R-RESCUE-VentilationLignade R14
@@
 F 0 "#PWR045" H 5200 660 30  0001 C CNN
 F 1 "+3.3V" H 5200 810 30  0000 C CNN
-F 2 "" H 5200 700 60  0000 C CNN
-F 3 "" H 5200 700 60  0000 C CNN
+F 2 "" H 5200 700 60  0001 C CNN
+F 3 "" H 5200 700 60  0001 C CNN
 	1    5200 700
 	1    0    0    -1
@@
 F 0 "#PWR046" H 4650 3450 30  0001 C CNN
 F 1 "GND" H 4650 3380 30  0001 C CNN
-F 2 "" H 4650 3450 60  0000 C CNN
-F 3 "" H 4650 3450 60  0000 C CNN
+F 2 "" H 4650 3450 60  0001 C CNN
+F 3 "" H 4650 3450 60  0001 C CNN
 	1    4650 3450
 	1    0    0    -1
@@
 F 0 "#PWR047" H 4950 2650 30  0001 C CNN
 F 1 "GND" H 4950 2580 30  0001 C CNN
-F 2 "" H 4950 2650 60  0000 C CNN
-F 3 "" H 4950 2650 60  0000 C CNN
+F 2 "" H 4950 2650 60  0001 C CNN
+F 3 "" H 4950 2650 60  0001 C CNN
 	1    4950 2650
 	1    0    0    -1
@@
 Connection ~ 4700 2550
 Wire Wire Line
-	4650 3150 4650 3450
+	4650 3450 4650 3150
 $Comp
 L R-RESCUE-VentilationLignade R15
@@
 F 0 "#PWR048" H 5200 2060 30  0001 C CNN
 F 1 "+3.3V" H 5200 2210 30  0000 C CNN
-F 2 "" H 5200 2100 60  0000 C CNN
-F 3 "" H 5200 2100 60  0000 C CNN
+F 2 "" H 5200 2100 60  0001 C CNN
+F 3 "" H 5200 2100 60  0001 C CNN
 	1    5200 2100
 	1    0    0    -1
@@
 F 0 "#PWR049" H 4650 4800 30  0001 C CNN
 F 1 "GND" H 4650 4730 30  0001 C CNN
-F 2 "" H 4650 4800 60  0000 C CNN
-F 3 "" H 4650 4800 60  0000 C CNN
+F 2 "" H 4650 4800 60  0001 C CNN
+F 3 "" H 4650 4800 60  0001 C CNN
 	1    4650 4800
 	1    0    0    -1
@@
 F 0 "#PWR050" H 4950 4000 30  0001 C CNN
 F 1 "GND" H 4950 3930 30  0001 C CNN
-F 2 "" H 4950 4000 60  0000 C CNN
-F 3 "" H 4950 4000 60  0000 C CNN
+F 2 "" H 4950 4000 60  0001 C CNN
+F 3 "" H 4950 4000 60  0001 C CNN
 	1    4950 4000
 	1    0    0    -1
@@
 Connection ~ 4700 3900
 Wire Wire Line
-	4650 4500 4650 4800
+	4650 4800 4650 4500
 $Comp
 L R-RESCUE-VentilationLignade R16
@@
 F 0 "#PWR051" H 5200 3410 30  0001 C CNN
 F 1 "+3.3V" H 5200 3560 30  0000 C CNN
-F 2 "" H 5200 3450 60  0000 C CNN
-F 3 "" H 5200 3450 60  0000 C CNN
+F 2 "" H 5200 3450 60  0001 C CNN
+F 3 "" H 5200 3450 60  0001 C CNN
 	1    5200 3450
 	1    0    0    -1
@@
 F 0 "#PWR052" H 4650 6200 30  0001 C CNN
 F 1 "GND" H 4650 6130 30  0001 C CNN
-F 2 "" H 4650 6200 60  0000 C CNN
-F 3 "" H 4650 6200 60  0000 C CNN
+F 2 "" H 4650 6200 60  0001 C CNN
+F 3 "" H 4650 6200 60  0001 C CNN
 	1    4650 6200
 	1    0    0    -1
@@
 F 0 "#PWR053" H 4950 5400 30  0001 C CNN
 F 1 "GND" H 4950 5330 30  0001 C CNN
-F 2 "" H 4950 5400 60  0000 C CNN
-F 3 "" H 4950 5400 60  0000 C CNN
+F 2 "" H 4950 5400 60  0001 C CNN
+F 3 "" H 4950 5400 60  0001 C CNN
 	1    4950 5400
 	1    0    0    -1
@@
 F 0 "#PWR054" H 5200 4810 30  0001 C CNN
 F 1 "+3.3V" H 5200 4960 30  0000 C CNN
-F 2 "" H 5200 4850 60  0000 C CNN
-F 3 "" H 5200 4850 60  0000 C CNN
+F 2 "" H 5200 4850 60  0001 C CNN
+F 3 "" H 5200 4850 60  0001 C CNN
 	1    5200 4850
 	1    0    0    -1
@@
 Connection ~ 5200 5600
 Wire Wire Line
-	4650 5900 4650 6200
+	4650 6200 4650 5900
 $Comp
 L OPTO-TRANSISTOR-RESCUE-VentilationLignade U6
@@
 F 0 "#PWR055" H 4650 7600 30  0001 C CNN
 F 1 "GND" H 4650 7530 30  0001 C CNN
-F 2 "" H 4650 7600 60  0000 C CNN
-F 3 "" H 4650 7600 60  0000 C CNN
+F 2 "" H 4650 7600 60  0001 C CNN
+F 3 "" H 4650 7600 60  0001 C CNN
 	1    4650 7600
 	1    0    0    -1
@@
 F 0 "#PWR056" H 4950 6800 30  0001 C CNN
 F 1 "GND" H 4950 6730 30  0001 C CNN
-F 2 "" H 4950 6800 60  0000 C CNN
-F 3 "" H 4950 6800 60  0000 C CNN
+F 2 "" H 4950 6800 60  0001 C CNN
+F 3 "" H 4950 6800 60  0001 C CNN
 	1    4950 6800
 	1    0    0    -1
@@
 Connection ~ 4700 6700
 Wire Wire Line
-	4650 7300 4650 7600
+	4650 7600 4650 7300
 $Comp
 L R-RESCUE-VentilationLignade R18
@@
 F 0 "#PWR057" H 5200 6210 30  0001 C CNN
 F 1 "+3.3V" H 5200 6360 30  0000 C CNN
-F 2 "" H 5200 6250 60  0000 C CNN
-F 3 "" H 5200 6250 60  0000 C CNN
+F 2 "" H 5200 6250 60  0001 C CNN
+F 3 "" H 5200 6250 60  0001 C CNN
 	1    5200 6250
 	1    0    0    -1
@@
 F 0 "#PWR058" H 2500 7700 40  0001 C CNN
 F 1 "GNDPWR" H 2500 7570 40  0000 C CNN
-F 2 "" H 2500 7650 60  0000 C CNN
-F 3 "" H 2500 7650 60  0000 C CNN
+F 2 "" H 2500 7650 60  0001 C CNN
+F 3 "" H 2500 7650 60  0001 C CNN
 	1    2500 7650
 	1    0    0    -1
@@
 	3800 1750 3950 1750
 Wire Wire Line
-	4450 1750 4650 1750
+	4650 1750 4450 1750
 $Comp
 L R-RESCUE-VentilationLignade R20
@@
 	3800 3150 3950 3150
 Wire Wire Line
-	4450 3150 4650 3150
+	4650 3150 4450 3150
 $Comp
 L R-RESCUE-VentilationLignade R21
@@
 $EndComp
 Wire Wire Line
-	4450 4500 4650 4500
+	4650 4500 4450 4500
 $Comp
 L R-RESCUE-VentilationLignade R22
@@
 	3800 5900 3950 5900
 Wire Wire Line
-	4450 5900 4650 5900
+	4650 5900 4450 5900
 $Comp
 L R-RESCUE-VentilationLignade R23
@@
 $EndComp
 Wire Wire Line
-	4450 7300 4650 7300
+	4650 7300 4450 7300
 Wire Wire Line
 	3800 4500 3950 4500
